File: RetroPanel Module/smart_switch.sch (KiCad schematic (older format))
At the start: 11 parts, among them J12 +5VSB, J13 PWR_ON, J14 PWR_OK, J15 COMMON, U2 NE555P

Commit message: Small tweaks
Other:
- note added: "Note that the colours assigned in the specification\nmight not actually match the cable that you have,\nin particular the cheap extensions and ATX to AT\ncable harnesses may have shuffled these around\ndepending on what they had on hand."
- moved on the sheet: C6, C7, C8, J12, J13, J14, J15, R18, R19, R20, U2

Commit message: Moved power diode
Other:
- note added: "(Black)"
- note added: "(Purple)"
- note removed: "(BLACK)"
Changed lines of the file:
@@
 $EndComp
 Text Notes 7350 5025 0    50   ~ 0
-(BLACK)
+(Black)
 Text Notes 7350 3675 0    50   ~ 0
 (Green)
@@
 $EndComp
 Text Notes 7350 3075 0    50   ~ 0
-(Grey)
+(Purple)
 $Comp
 L Timer:NE555P U2

Commit message: Small tweaks
Parts:
- C7: footprint RetroPanel:CP_Radial_D4.0mm_P2.00mm_Custom -> Capacitor_THT:CP_Radial_D4.0mm_P2.00mm
Changed lines of the file:
@@
 F 0 "C7" H 6363 4871 50  0000 L CNN
 F 1 "4.7uF" H 6363 4780 50  0000 L CNN
-F 2 "RetroPanel:CP_Radial_D4.0mm_P2.00mm_Custom" H 6275 4825 50  0001 C CNN
+F 2 "Capacitor_THT:CP_Radial_D4.0mm_P2.00mm" H 6275 4825 50  0001 C CNN
 F 3 "~" H 6275 4825 50  0001 C CNN
 	1    6275 4825

Commit message: Better description for CA display usage
Other:
- note added: "Note that the colours assigned in the specification\nmight not actually match the cable that you have,\nin particular the cheap extensions and ATX to AT\ncable harnesses may have shuffled these around\ndepending on what they had on hand. Usually you\ncan find the correct orientation when looking at \nthe three orange 3.3v cables clustered together at\nthe top.\n\nThe easiest way to create the nec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"
- note removed: "Note that the colours assigned in the specification\nmight not actually match the cable that you have,\nin particular the cheap extensions and ATX to AT\ncable harnesses may have shuffled these around\ndepending on what they had on hand."
Changed lines of the file:
@@
 Comp ""
 Comment1 ""
-Comment2 "latching switch is installed on the front and then wired to the ATX to AT cables."
+Comment2 "latching switch can be installed on the front and then wired to the ATX to AT cables."
 Comment3 "to shut down when one of its outputs have been shorted. If the circuit is not needed, a"
 Comment4 "Circuit for using standard ATX-case with ATX to AT-kits, the circuit allows the PSU "
@@
 	1    0    0    -1
 $EndComp
-Text Notes 7800 3225 0    50   ~ 0
-Note that the colours assigned in the specification\nmight not actually match the cable that you have,\nin particular the cheap extensions and ATX to AT\ncable harnesses may have shuffled these around\ndepending on what they had on hand.
+Text Notes 7800 4125 0    50   ~ 0
+Note that the colours assigned in the specification\nmight not actually match the cable that you have,\nin particular the cheap extensions and ATX to AT\ncable harnesses may have shuffled these around\ndepending on what they had on hand. Usually you\ncan find the correct orientation when looking at \nthe three orange 3.3v cables clustered together at\nthe top.\n\nThe easiest way to create the necessary cable\nis to purchase both a cheap ATX-extension cable\nas well as an ATX to AT converter cable. You should\nalready have the black and green pigtail, the purple\none can be stolen directly from the extension. The\ngrey cable needs to be spliced because it'll be going\nto both the switching circuit as well as the MB.
 $EndSCHEMATC

Commit message: Optional standby power LED
Parts:
- added D2: STANDBY, LED_THT:LED_D5.0mm, symbol Device:LED
- added R22: 470, resistor:R_Axial_DIN0207_L6.3mm_D2.5mm_P10.16mm_Horizontal, symbol Device:R_Small
Connections:
- net +5VSB: now also D2.2 (A)
- net GND: now also R22.1
- new net: D2.1 (K), R22.2
Changed lines of the file:
@@
 Text Notes 7800 4125 0    50   ~ 0
 Note that the colours assigned in the specification\nmight not actually match the cable that you have,\nin particular the cheap extensions and ATX to AT\ncable harnesses may have shuffled these around\ndepending on what they had on hand. Usually you\ncan find the correct orientation when looking at \nthe three orange 3.3v cables clustered together at\nthe top.\n\nThe easiest way to create the necessary cable\nis to purchase both a cheap ATX-extension cable\nas well as an ATX to AT converter cable. You should\nalready have the black and green pigtail, the purple\none can be stolen directly from the extension. The\ngrey cable needs to be spliced because it'll be going\nto both the switching circuit as well as the MB.
+$Comp
+L Device:R_Small R?
+U 1 1 6379EE4C
+P 3725 3525
+AR Path="/6379EE4C" Ref="R?"  Part="1"
+AR Path="/63655027/6379EE4C" Ref="R22"  Part="1"
+F 0 "R22" H 3775 3475 50  0000 L CNN
+F 1 "470" H 3775 3550 50  0000 L CNN
+F 2 "resistor:R_Axial_DIN0207_L6.3mm_D2.5mm_P10.16mm_Horizontal" H 3725 3525 50  0001 C CNN
+F 3 "~" H 3725 3525 50  0001 C CNN
+	1    3725 3525
+	1    0    0    1
+$EndComp
+$Comp
+L power:GND #PWR0109
+U 1 1 6379FCF1
+P 3725 3625
+F 0 "#PWR0109" H 3725 3375 50  0001 C CNN
+F 1 "GND" H 3730 3452 50  0000 C CNN
+F 2 "" H 3725 3625 50  0001 C CNN
+F 3 "" H 3725 3625 50  0001 C CNN
+	1    3725 3625
+	1    0    0    -1
+$EndComp
+$Comp
+L Device:LED D2
+U 1 1 637A2E72
+P 3725 3200
+F 0 "D2" V 3764 3082 50  0000 R CNN
+F 1 "STANDBY" V 3673 3082 50  0000 R CNN
+F 2 "LED_THT:LED_D5.0mm" H 3725 3200 50  0001 C CNN
+F 3 "~" H 3725 3200 50  0001 C CNN
+	1    3725 3200
+	0    -1   -1   0
+$EndComp
+Wire Wire Line
+	3725 3425 3725 3350
+Wire Wire Line
+	3725 3050 3725 2900
+Wire Wire Line
+	3725 2900 4250 2900
+Connection ~ 4250 2900
 $EndSCHEMATC
