File: RetroPanel Side/RetroPanel Side.sch (KiCad schematic (older format))
At the start: 13 parts, among them M1 Mounting_Pin, M10 Mounting_Pad, M11 Mounting_Pad, M12 Mounting_Pad, M13 Mounting_Pad, M2 Mounting_Pin, M3 Mounting_Pin, M4 Mounting_Pad, M5 Mounting_Pad, M6 Mounting_Pad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

Commit message: Adjustable mounting with huge pads
Parts:
- added M14: Mounting_Pad, RetroPanel:Pad_pin, symbol mounting:Mounting_Pad
- M1: footprint mounting:M3_pin -> mounting:M3_adjustable
- M2: footprint mounting:M3_pin -> mounting:M3_big
Connections:
- net GND: now also M14.1
Changed lines of the file:
@@
 F 0 "M1" H 10850 675 50  0001 C CNN
 F 1 "Mounting_Pin" H 10850 500 50  0001 C CNN
-F 2 "mounting:M3_pin" H 10850 575 50  0001 C CNN
+F 2 "mounting:M3_adjustable" H 10850 575 50  0001 C CNN
 F 3 "~" H 10850 575 50  0001 C CNN
 	1    10850 575
@@
 F 0 "M2" H 10975 675 50  0001 C CNN
 F 1 "Mounting_Pin" H 10975 500 50  0001 C CNN
-F 2 "mounting:M3_pin" H 10975 575 50  0001 C CNN
+F 2 "mounting:M3_big" H 10975 575 50  0001 C CNN
 F 3 "~" H 10975 575 50  0001 C CNN
 	1    10975 575
@@
 	1    0    0    -1
 $EndComp
+$Comp
+L mounting:Mounting_Pad M14
+U 1 1 636EFA56
+P 9725 950
+F 0 "M14" H 9725 1050 50  0001 C CNN
+F 1 "Mounting_Pad" H 9725 875 50  0001 C CNN
+F 2 "RetroPanel:Pad_pin" H 9725 950 50  0001 C CNN
+F 3 "~" H 9725 950 50  0001 C CNN
+	1    9725 950
+	1    0    0    -1
+$EndComp
+Wire Wire Line
+	9725 1100 9725 1175
+Wire Wire Line
+	9725 1175 9850 1175
+Connection ~ 9850 1175
 $EndSCHEMATC

Commit message: Fixed RS-232 connector and export files for second prototype
Parts:
- added M15: Mounting_Pin, mounting:M3_pin_wide, symbol mounting:Mounting_Pin
Connections:
- net GND: now also M15.1
Changed lines of the file:
@@
 L power:PWR_FLAG #FLG0101
 U 1 1 63693A74
-P 10775 800
-F 0 "#FLG0101" H 10775 875 50  0001 C CNN
-F 1 "PWR_FLAG" V 10775 927 50  0001 L CNN
-F 2 "" H 10775 800 50  0001 C CNN
-F 3 "~" H 10775 800 50  0001 C CNN
-	1    10775 800
+P 10650 800
+F 0 "#FLG0101" H 10650 875 50  0001 C CNN
+F 1 "PWR_FLAG" V 10650 927 50  0001 L CNN
+F 2 "" H 10650 800 50  0001 C CNN
+F 3 "~" H 10650 800 50  0001 C CNN
+	1    10650 800
 	0    -1   -1   0
 $EndComp
@@
 	10600 1175 10725 1175
 Connection ~ 11100 800
-Wire Wire Line
-	10775 800  10850 800
 Connection ~ 10850 800
 $Comp
@@
 	9725 1175 9850 1175
 Connection ~ 9850 1175
+$Comp
+L mounting:Mounting_Pin M15
+U 1 1 63701E78
+P 10725 575
+F 0 "M15" H 10725 675 50  0001 C CNN
+F 1 "Mounting_Pin" H 10725 500 50  0001 C CNN
+F 2 "mounting:M3_pin_wide" H 10725 575 50  0001 C CNN
+F 3 "~" H 10725 575 50  0001 C CNN
+	1    10725 575
+	1    0    0    -1
+$EndComp
+Wire Wire Line
+	10725 725  10725 800
+Wire Wire Line
+	10725 800  10850 800
+Wire Wire Line
+	10725 800  10650 800
+Connection ~ 10725 800
 $EndSCHEMATC
