File: RetroPanel SD35VC0/RetroPanel SD35VC0.kicad_pcb (KiCad board)
At the start: 2 copper layers, 100 x 97.9 mm, 22 parts, among them J1 Front Panel, J2 SD35VC0, J3 IDE, J4 GND, J5 +5V, J7 POWER, M1 Mounting_Pin, M10 Mounting_Pad, M11 Mounting_Pad, M12 Mounting_Pad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

Commit message: SD35VC0 Front sketched out
Parts:
- added J10: LED_POWER, RetroPanel:PinHeader_1x02_P2.54mm_Vertical, F.Cu at (171.6, 63.2)
- added J6: SW_TURBO, RetroPanel:PinHeader_1x02_P2.54mm_Vertical, F.Cu at (179.2, 56.8)
- added J8: LED_TURBO, RetroPanel:PinHeader_1x02_P2.54mm_Vertical, F.Cu at (179.2, 63.2)
- added J9: SW_POWER, RetroPanel:PinHeader_1x02_P2.54mm_Vertical, F.Cu at (171.6, 56.8)
- added R1: 0, resistor:R_Axial_DIN0207_L6.3mm_D2.5mm_P10.16mm_Horizontal, F.Cu at (163.9, 57.4)
- added R2: 0, resistor:R_Axial_DIN0207_L6.3mm_D2.5mm_P10.16mm_Horizontal, F.Cu at (163.9, 61.3)
- J1: footprint RetroPanel:Module_Panel -> RetroPanel:SD35VC0_Module_Panel
- turned M14 to 270 degrees
Connections:
- J1 pad 1: (no net) -> GND
- J1 pad 22: (no net) -> LED_TURBO1
- J1 pad 23: (no net) -> LED_TURBO2
- J1 pad 24: (no net) -> SW_TURBO1
- J1 pad 25: (no net) -> SW_TURBO2
- J1 pad 30: GND -> +5V
- J1 pad 6: (no net) -> SW_PWR1
- J1 pad 7: (no net) -> SW_PWR2
- J1 pad 8: (no net) -> LED_PWR1
- J1 pad 9: (no net) -> LED_PWR2
- J5 pad 1: Net-(J5-Pad1) -> +5V
- J7 pad 4: Net-(J5-Pad1) -> +5V
Routing:
- net SW_TURBO1: track 0.00 -> 138.8 mm
- net SW_TURBO2: track 0.00 -> 136.5 mm, vias 0 -> 1
- net LED_TURBO2: track 0.00 -> 114.8 mm
- net LED_TURBO1: track 0.00 -> 95.5 mm
- net LED_PWR2: track 0.00 -> 85.4 mm
- net SW_PWR1: track 0.00 -> 78.0 mm
- net SW_PWR2: track 0.00 -> 76.7 mm
- net +5V: track 0.00 -> 76.0 mm
- net LED_PWR1: track 0.00 -> 56.1 mm, vias 0 -> 1
- net Net-(J5-Pad1): track 53.8 -> 0.00 mm
- net Net-(J8-Pad1): track 0.00 -> 19.8 mm
- net Net-(J10-Pad1): track 0.00 -> 9.15 mm
Other:
- board text added: "LED_POWER"
- board text added: "LED_TURBO"

Commit message: Changed SW_PWR to pads for cable as it probably should be
Parts:
- removed J9: SW_POWER, RetroPanel:PinHeader_1x02_P2.54mm_Vertical
- added J11: PWR_ON, RetroPanel:PSU_Wire, F.Cu at (197.0, 139.4)
- added J12: COMMON, RetroPanel:PSU_Wire, F.Cu at (198.2, 143.8)
- moved J10 15.9 mm to (187.4, 63.2)
- moved J7 8.52 mm to (191.0, 132.9)
- moved R1 7.75 mm to (168.4, 63.8)
- moved R2 5.12 mm to (168.4, 58.7)
Connections:
- J1 pad 7: SW_PWR2 -> GND
Routing:
- net SW_PWR2: track 76.7 -> 0.00 mm
- net SW_PWR1: track 78.0 -> 149.8 mm, vias 0 -> 2
- net Net-(J10-Pad1): track 9.15 -> 23.1 mm
- net +5V: track 76.0 -> 86.2 mm
- net LED_PWR1: track 56.1 -> 63.1 mm, vias 1 -> 0
- net Net-(J8-Pad1): track 19.8 -> 13.4 mm
- net LED_PWR2: track 85.4 -> 91.1 mm
- net GND: track 51.1 -> 53.8 mm
- net SW_TURBO1: track 138.8 -> 140.9 mm
- net LED_TURBO1: track 95.5 -> 93.6 mm
- net SW_TURBO2: track 136.5 -> 138.2 mm
